File: power-rj45.kicad_pcb (KiCad board)
At the start: 4 copper layers, 73.5 x 20 mm, 42 parts, among them J101 2x05_Horizontal, J102 NE8FAH, J103 JAE_DX07S016JA3, J104 2x05_Horizontal, J105 NE8FAH, J106 WAGO-2065, J107 WAGO-2065, J108 WAGO-2065, J109 WAGO-2065, Q201 BSC010N04LS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

Commit message: Update icons
Parts:
- removed ICON101, ICON104: Minus, V2_Artwork:Minus_Small
- added ICON110: Arrow_Out, V2_Artwork:Arrow_Out, F.Cu at (131.2, 99.0)
- added ICON111: Arrow_Out, V2_Artwork:Arrow_Out, F.Cu at (176.2, 99.0)
Connections:
- J103 pad V: unconnected-(J103-VBUS-PadV) -> VBUS
Routing:
- net unconnected-(J103-VBUS-PadV): track 6.00 -> 0.00 mm, vias 2 -> 0
- net VBUS: track 0.00 -> 5.94 mm, vias 0 -> 2

Commit message: Replace icons
Parts:
- removed ICON108: Socket, V2_Artwork:Socket_Small
- removed ICON109: Plug, V2_Artwork:Plug_Small
- added ICON101: Arrow_In, V2_Artwork:Arrow_In, F.Cu at (123.5, 113.8)
- added ICON104: Arrow_Out, V2_Artwork:Arrow_Out, F.Cu at (184.0, 113.8)

Commit message: Update icons
Parts:
- moved ICON101 60.5 mm to (184.0, 113.8), turned to 180 degrees
- moved ICON104 60.2 mm to (123.8, 113.8), turned to 180 degrees
Changed lines of the file:
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@@
 	(footprint "V2_Artwork:Arrow_In"
 		(layer "F.Cu")
-		(at 123.5 113.75)
+		(at 184 113.75 180)
 		(property "Reference" "ICON101"
-			(at 0 -2.5 0)
+			(at 0 -2.5 180)
 			(unlocked yes)
 			(layer "F.SilkS")
@@
 		)
 		(property "Value" "Arrow_In"
-			(at 0 2.5 0)
+			(at 0 2.5 180)
 			(unlocked yes)
 			(layer "F.Fab")
@@
 		)
 		(property "Footprint" "V2_Artwork:Arrow_In"
-			(at 0 0 0)
+			(at 0 0 180)
 			(unlocked yes)
 			(layer "F.Fab")
@@
 		)
 		(property "Datasheet" ""
-			(at 0 0 0)
+			(at 0 0 180)
 			(unlocked yes)
 			(layer "F.Fab")
@@
 		)
 		(property "Description" ""
-			(at 0 0 0)
+			(at 0 0 180)
 			(unlocked yes)
 			(layer "F.Fab")
@@
 		)
 		(property "Sim.Enable" "0"
-			(at 0 0 0)
+			(at 0 0 180)
 			(unlocked yes)
 			(layer "F.Fab")
@@
 	(footprint "V2_Artwork:Arrow_Out"
 		(layer "F.Cu")
-		(at 184 113.75)
+		(at 123.75 113.75 180)
 		(property "Reference" "ICON104"
-			(at 0 -2.5 0)
+			(at 0 -2.5 180)
 			(unlocked yes)
 			(layer "F.SilkS")
@@
 		)
 		(property "Value" "Arrow_Out"
-			(at 0 2.5 0)
+			(at 0 2.5 180)
 			(unlocked yes)
 			(layer "F.Fab")
@@
 		)
 		(property "Footprint" "V2_Artwork:Arrow_Out"
-			(at 0 0 0)
+			(at 0 0 180)
 			(unlocked yes)
 			(layer "F.Fab")
@@
 		)
 		(property "Datasheet" ""
-			(at 0 0 0)
+			(at 0 0 180)
 			(unlocked yes)
 			(layer "F.Fab")
@@
 		)
 		(property "Description" ""
-			(at 0 0 0)
+			(at 0 0 180)
 			(unlocked yes)
 			(layer "F.Fab")
@@
 		)
 		(property "Sim.Enable" "0"
-			(at 0 0 0)
+			(at 0 0 180)
 			(unlocked yes)
 			(layer "F.Fab")
