File: connector-poe.kicad_pcb (KiCad board)
At the start: 4 copper layers, 73.5 x 20 mm, 42 parts, among them J101 2x05_Horizontal, J102 NE8FAH, J103 JAE_DX07S016JA3, J104 2x05_Horizontal, J105 NE8FAH, J106 WAGO-2065, J107 WAGO-2065, J108 WAGO-2065, J109 WAGO-2065, Q201 BSC010N04LS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

Commit message: Refresh
Parts:
- moved ICON104 3.26 mm to (120.5, 113.5)
- moved ICON101 3.01 mm to (187.0, 113.5)
- moved ICON106 0.71 mm to (175.8, 96.8)
- moved ICON103 0.50 mm to (179.2, 98.5)
- moved ICON105 0.50 mm to (128.2, 102.0)
- moved ICON107 0.50 mm to (131.2, 96.8)
- moved ICON111 0.50 mm to (175.8, 99.0)
Connections:
- C102 pad 1: /+24V-Input -> /+24V-Supply
- C201 pad 1: /+24V-Input -> /+24V-Supply
- C301 pad 1: /+24V-Supply -> +24V
- C302 pad 1: /+24V-Supply -> +24V
- J102 pad 4: /+24V-Input -> /+24V-Supply
- J102 pad 5: /+24V-Input -> /+24V-Supply
- J105 pad 4: /+24V-Input -> /+24V-Supply
- J105 pad 5: /+24V-Input -> /+24V-Supply
- J106 pad 1: /+24V-Supply -> +24V
- Q201 pad 1: /+24V-Supply -> +24V
- Q201 pad 5: /+24V-Input -> /+24V-Supply
- R201 pad 1: /+24V-Input -> /+24V-Supply
- TVS101 pad 2: /+24V-Input -> /+24V-Supply
- U201 pad 1: /+24V-Input -> /+24V-Supply
- U201 pad 5: /+24V-Input -> /+24V-Supply
- U201 pad 8: /+24V-Supply -> +24V
- U301 pad 2: /+24V-Supply -> +24V
- U301 pad 3: /+24V-Supply -> +24V
Routing:
- net /+24V-Input: track 15.2 -> 0.00 mm
- net /+24V-Supply: track 3.19 -> 15.2 mm, vias 16 -> 0
- net +24V: track 0.00 -> 3.19 mm, vias 0 -> 16
- added copper zone on B.Cu, net +24V
- added copper zone on F.Cu, net +24V
- added copper zone on In1.Cu, net /+24V-Supply
- added copper zone on In2.Cu, net /+24V-Supply
- removed copper zone on B.Cu, net /+24V-Input
- removed copper zone on F.Cu, net /+24V-Input
- removed copper zone on In1.Cu, net /+24V-Input
- removed copper zone on In2.Cu, net /+24V-Input
