File: connector-poe.kicad_sch (KiCad schematic)
At the start: 29 parts, among them J101 2x05_Horizontal, J102 NE8FAH, J103 JAE_DX07S016JA3, J104 2x05_Horizontal, J105 NE8FAH, J106 WAGO-2065, J107 WAGO-2065, J108 WAGO-2065, J109 WAGO-2065

Commit message: Refresh
Connections:
- net +24V-Input is gone; now on net +24V-Supply: C102.1, J102.4, J102.5, J105.4, J105.5, TVS101.2 (A)
- net +24V-Supply: no longer J106.1
- new net +24V: J106.1
Other:
- note added: "Polarity Protection / +5V Power"
- note added: "V2 Link / PoE Mode B"
- note removed: "+5V Power"
- note removed: "V2 Link"
- moved on the sheet: C102, J106, J107, J108, J109, TVS101
