File: connector-poe.kicad_sch (KiCad schematic)
At the start: 27 parts, among them J101 2x05_Horizontal, J102 NE8FAH, J103 JAE_DX07S016JA3, J104 2x05_Horizontal, J105 NE8FAH, J106 WAGO-2065, J107 WAGO-2065, J108 WAGO-2065, J109 WAGO-2065

Commit message: Resize to 70 mm
Parts:
- ICON102: footprint V2_Artwork:Logo_Small -> V2_Artwork:Logo_Tiny
- renumbered C102 to C101, ICON106 to ICON101, ICON107 to ICON104, ICON101 to ICON106, ICON104 to ICON107, J108 to J107, J107 to J108
Connections:
- net RJ45-Shield renamed Shield
Other:
- note added: "V2 Link – PoE Mode B"
- note removed: "V2 Link / PoE Mode B"
